File: CANoBUS.kicad_sch (KiCad schematic)
At the start: 3 parts, among them J1 USB_B_Mini, U1 ATSAMD11D14A-M, Y1 Crystal_GND24_Small

Commit message: wip
Parts:
- added ARM_DEBUGGER: Conn_02x05_Odd_Even, symbol Connector_Generic:Conn_02x05_Odd_Even
- added C1, C2: 100nF, symbol Device:C
- added C10: 10uF, symbol Device:C
- added C3: 4.7uF, symbol Device:C
- added C4, C5: 12pF, symbol Device:C
- added D1: PRTR5V0U2X, Package_TO_SOT_SMD:SOT-143, symbol Power_Protection:PRTR5V0U2X
- added FB1: FerriteBead, symbol Device:FerriteBead
- added R10: 100k, symbol Device:R
- added R20: 10k, symbol Device:R
- added R21: 47, symbol Device:R
- added R23, R24: 0, symbol Device:R
- added SW1: SW_Push, symbol Switch:SW_Push
- added U2: MIC5504-3.3YM5, Package_TO_SOT_SMD:SOT-23-5, symbol Regulator_Linear:MIC5504-3.3YM5
- Y1: footprint (none) -> Crystal:Crystal_SMD_3225-4Pin_3.2x2.5mm
Connections:
- net RX: now reaches U1.10 (PA11)
- net SDA: now reaches U1.15 (PA22)
- net SCL: now reaches U1.16 (PA23)
- net RESET: now reaches U1.18 (PA28/~{RST})
- net RESET: now also C1.1, R20.1, R21.2
- net SWCLK: now reaches U1.19 (PA30/SWCLK)
- net SWCLK: now also ARM_DEBUGGER.4 (Pin_4)
- net SWDIO: now reaches U1.20 (PA31/SWDIO)
- net SWDIO: now also ARM_DEBUGGER.2 (Pin_2)
- net GND: now reaches U1.23 (GND)
- net GND: now also J1.5 (GND), J1.6 (Shield), Y1.2, Y1.4, ARM_DEBUGGER.3 (Pin_3), ARM_DEBUGGER.5 (Pin_5), ARM_DEBUGGER.9 (Pin_9), C1.2, C10.2, C2.2, C3.2, C4.2, C5.2, D1.1 (GND), SW1.1, U2.2 (GND)
- net +3.3V: now reaches U1.24 (VDD)
- net +3.3V: now also ARM_DEBUGGER.1 (Pin_1), C2.1, C3.1, R20.2, U2.5 (VOUT)
- net MOSI: now reaches U1.5 (PA06)
- net SCK: now reaches U1.6 (PA07)
- net SS: now reaches U1.7 (PA08/XIN)
- net MISO: now reaches U1.8 (PA09/XOUT)
- net TX: now reaches U1.9 (PA10)
- net XTAL+: now reaches Y1.1
- net XTAL+: now also C4.1
- net XTAL-: now reaches Y1.3
- net XTAL-: now also C5.1
- net at J1.1 (VBUS): now also FB1.1
- net D-: now reaches J1.2 (D-)
- net D-: now also D1.3 (I/O2), R24.2
- net D+: now reaches J1.3 (D+)
- net D+: now also D1.2 (I/O1), R23.2
- net USB_N renamed DN
- net DN: now also R24.1
- net USB_P: no longer names the net of U1.22 (PA25)
- new net: R21.1, SW1.2
- new net: C10.1, R10.1, U2.3 (EN)
- new net DP: R23.1
- new net EXT_RESET: ARM_DEBUGGER.10 (Pin_10)
- new net VBUS: D1.4 (VCC), FB1.2, R10.2, U2.1 (VIN)
- no-connect marks 0 -> 4
Other:
- moved on the sheet: U1, Y1
